File: boards/ECE 445 - Suction Sense PCB-1.kicad_pcb (KiCad board)
At the start: 2 copper layers, 92.7 x 88.9 mm, 48 parts, among them J1 Paddle Sensor, J2 Motion Sensor, J3 Battery Connector, J4 Barrel_Jack, J5 Conn_01x06_Pin, U1 ESP32-WROOM-32E, U2 TPS2121RUXR, U3 AP62150Z6, U4 MCP73831-2-OT, U5 TPS613222ADBVR

Commit message: new upadtes to board
Parts:
- L2: value L -> 2.2uH
Connections:
- D1 pad 2: GND -> (no net)
- R4 pad 1: GND -> (no net)
Routing:
- net /5vA: track 5.36 -> 40.8 mm, vias 0 -> 2
- net GND: track 48.2 -> 40.9 mm, vias 9 -> 7
Changed lines of the file:
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@@
 			)
 		)
-		(property "Value" "L"
+		(property "Value" "2.2uH"
 			(at 0 1.75 90)
 			(layer "F.Fab")
@@
 			(layers "F.Cu" "F.Mask" "F.Paste")
 			(roundrect_rratio 0.208333)
-			(net 2 "GND")
 			(pintype "passive")
 		)
@@
 			(layers "F.Cu" "F.Mask" "F.Paste")
 			(roundrect_rratio 0.25)
-			(net 2 "GND")
 			(pinfunction "A")
 			(pintype "passive")
@@
 	)
 	(segment
+		(start 104.8 65.5)
+		(end 104.361 65.939)
+		(width 0.2)
+		(layer "F.Cu")
+		(net 2)
+	)
+	(segment
 		(start 132.95 85.45)
 		(end 132.9 85.5)
@@
 	)
 	(segment
-		(start 104.7 65.5)
-		(end 104.762 65.5625)
-		(width 0.2)
-		(layer "F.Cu")
-		(net 2)
-	)
-	(segment
 		(start 130.6965 64.481)
 		(end 130.048 65.1295)
@@
 	)
 	(segment
-		(start 104.762 67.8317)
-		(end 104.762 70.1)
+		(start 130.048 65.1295)
+		(end 125.857 65.1295)
 		(width 0.2)
 		(layer "F.Cu")
@@
 	)
 	(segment
-		(start 130.048 65.1295)
-		(end 125.857 65.1295)
+		(start 104.5959 69.699)
+		(end 104.7625 69.699)
 		(width 0.2)
 		(layer "F.Cu")
@@
 	)
 	(segment
-		(start 104.762 65.5625)
-		(end 104.762 67.8312)
+		(start 104.7625 70.1)
+		(end 104.762 70.1)
 		(width 0.2)
 		(layer "F.Cu")
@@
 	)
 	(segment
-		(start 104.7625 70.1)
-		(end 104.762 70.1)
+		(start 104.361 65.939)
+		(end 104.361 69.4641)
 		(width 0.2)
 		(layer "F.Cu")
@@
 	)
 	(segment
-		(start 154.875 101)
-		(end 156.4 102.525)
-		(width 0.2)
-		(layer "F.Cu")
-		(net 2)
-	)
-	(segment
-		(start 104.8 65.5)
-		(end 104.7 65.5)
+		(start 104.361 69.4641)
+		(end 104.5959 69.699)
 		(width 0.2)
 		(layer "F.Cu")
@@
 	)
 	(segment
-		(start 104.762 67.8312)
-		(end 104.762 70.1)
+		(start 154.875 101)
+		(end 156.4 102.525)
 		(width 0.2)
 		(layer "F.Cu")
@@
 	)
 	(via
-		(at 114 66.6)
-		(size 0.6)
-		(drill 0.3)
-		(layers "F.Cu" "B.Cu")
-		(free yes)
-		(net 2)
-	)
-	(via
 		(at 160.9 103.3)
 		(size 0.6)
@@
 		(net 2)
 	)
-	(via
-		(at 115.1 62.1)
-		(size 0.6)
-		(drill 0.3)
-		(layers "F.Cu" "B.Cu")
-		(net 2)
-	)
-	(segment
-		(start 114 66.6)
-		(end 114 63.2)
-		(width 0.2)
-		(layer "B.Cu")
-		(net 2)
-	)
 	(segment
 		(start 128.4 90.1)
@@
 	)
 	(segment
-		(start 114 63.2)
-		(end 115.1 62.1)
-		(width 0.2)
-		(layer "B.Cu")
-		(net 2)
-	)
-	(segment
 		(start 160.8 103.4)
 		(end 160.9 103.3)
@@
 	)
 	(segment
-		(start 135.65 67.021)
-		(end 133.8715 67.021)
+		(start 127.35484 70.301)
+		(end 130.959 70.301)
 		(width 0.2)
 		(layer "F.Cu")
@@
 	)
 	(segment
-		(start 114.681 59.944)
-		(end 119.0685 64.3315)
+		(start 94.488 65.38234)
+		(end 99.92634 59.944)
 		(width 0.2)
 		(layer "F.Cu")
@@
 	)
 	(segment
-		(start 146.0471 70.9461)
-		(end 146.0471 75.799)
+		(start 135.65 67.021)
+		(end 133.8715 67.021)
 		(width 0.2)
 		(layer "F.Cu")
@@
 	)
 	(segment
-		(start 95.115 116.451)
-		(end 93.98 115.316)
+		(start 114.681 59.944)
+		(end 119.0685 64.3315)
 		(width 0.2)
 		(layer "F.Cu")
@@
 	)
 	(segment
-		(start 133.8715 67.021)
-		(end 133.35 67.5425)
+		(start 146.0471 70.9461)
+		(end 146.0471 75.799)
 		(width 0.2)
 		(layer "F.Cu")
@@
 	)
 	(segment
-		(start 93.98 115.316)
-		(end 93.98 65.89034)
+		(start 117.317 116.451)
+		(end 95.115 116.451)
 		(width 0.2)
 		(layer "F.Cu")
@@
 	)
 	(segment
-		(start 121.38534 64.3315)
-		(end 127.35484 70.301)
+		(start 133.8715 67.021)
+		(end 133.35 67.5425)
 		(width 0.2)
 		(layer "F.Cu")
@@
 	)
 	(segment
-		(start 134.239 67.021)
-		(end 135.65 67.021)
+		(start 142.122 67.021)
+		(end 146.0471 70.9461)
 		(width 0.2)
 		(layer "F.Cu")
@@
 	)
 	(segment
-		(start 142.122 67.021)
-		(end 146.0471 70.9461)
+		(start 149.733 87.757)
+		(end 149.606 87.884)
 		(width 0.2)
 		(layer "F.Cu")
@@
 	)
 	(segment
-		(start 149.733 87.757)
-		(end 149.606 87.884)
+		(start 134.239 67.021)
+		(end 135.65 67.021)
 		(width 0.2)
 		(layer "F.Cu")
@@
 	)
 	(segment
-		(start 127.35484 70.301)
-		(end 130.959 70.301)
+		(start 135.65 67.021)
+		(end 142.122 67.021)
 		(width 0.2)
 		(layer "F.Cu")
@@
 	)
 	(segment
-		(start 135.65 67.021)
-		(end 142.122 67.021)
+		(start 153.8141 83.566)
+		(end 155.321 83.566)
 		(width 0.2)
 		(layer "F.Cu")
@@
 	)
 	(segment
-		(start 117.317 116.451)
-		(end 95.115 116.451)
+		(start 119.0685 64.3315)
+		(end 121.38534 64.3315)
 		(width 0.2)
 		(layer "F.Cu")
@@
 	)
 	(segment
-		(start 153.8141 83.566)
-		(end 155.321 83.566)
+		(start 95.115 116.451)
+		(end 94.488 115.824)
 		(width 0.2)
 		(layer "F.Cu")
@@
 	)
 	(segment
-		(start 93.98 65.89034)
-		(end 99.92634 59.944)
+		(start 94.488 115.824)
+		(end 94.488 65.38234)
 		(width 0.2)
 		(layer "F.Cu")
@@
 	)
 	(segment
-		(start 119.0685 64.3315)
-		(end 121.38534 64.3315)
+		(start 121.38534 64.3315)
+		(end 127.35484 70.301)
 		(width 0.2)
 		(layer "F.Cu")
@@
 	)
 	(segment
+		(start 104.648 98.933)
+		(end 103.886 99.695)
+		(width 0.2)
+		(layer "F.Cu")
+		(net 53)
+	)
+	(segment
+		(start 104.648 75.52713)
+		(end 104.648 98.933)
+		(width 0.2)
+		(layer "F.Cu")
+		(net 53)
+	)
+	(segment
 		(start 103.8755 75.4245)
 		(end 104.013 75.287)
@@
 		(net 53)
 	)
+	(segment
+		(start 103.759 108.4365)
+		(end 102.235 109.9605)
+		(width 0.2)
+		(layer "F.Cu")
+		(net 53)
+	)
+	(segment
+		(start 103.759 105.029)
+		(end 103.759 108.4365)
+		(width 0.2)
+		(layer "F.Cu")
+		(net 53)
+	)
+	(via
+		(at 103.759 105.029)
+		(size 0.6)
+		(drill 0.3)
+		(layers "F.Cu" "B.Cu")
+		(net 53)
+	)
+	(via
+		(at 103.886 99.695)
+		(size 0.6)
+		(drill 0.3)
+		(layers "F.Cu" "B.Cu")
+		(net 53)
+	)
+	(segment
+		(start 103.759 99.822)
+		(end 103.759 105.029)
+		(width 0.2)
+		(layer "B.Cu")
+		(net 53)
+	)
+	(segment
+		(start 103.886 99.695)
+		(end 103.759 99.822)
+		(width 0.2)
+		(layer "B.Cu")
+		(net 53)
+	)
